Commit message: add in camera link

File: mybot_description/urdf/mybot.xacro (robot description, xacro)
@@ -68,3 +68,28 @@
 	<wheel lr="left" tY="-1"/>
 	<wheel lr="right" tY="1"/>
+	<joint name="camera_joint" type="fixed">
+	    <origin xyz="${-cameraSize+chassisLength/2} 0 ${cameraSize+wheelRadius+cameraSize/2}" rpy="0 0 0"/>
+	    <parent link="chassis"/>
+	    <child link="camera"/>
+	</joint>
+	<link name="camera">
+	  <collision>
+	    <origin xyz="0 0 0" rpy="0 0 0"/>
+	    <geometry>
+	      <box size="${cameraSize} ${cameraSize} ${cameraSize}"/>
+	    </geometry>
+	  </collision>
+	  <visual>
+	    <origin xyz="0 0 0" rpy="0 0 0"/>
+	    <geometry>
+	      <box size="${cameraSize} ${cameraSize} ${cameraSize}"/>
+	    </geometry>
+	    <material name="blue"/>
+	  </visual>
+	  <inertial>
+	    <mass value="${cameraMass}" />
+	    <origin xyz="0 0 0" rpy="0 0 0"/>
+	    <box_inertia m="${cameraMass}" x="${cameraSize}" y="${cameraSize}" z="${cameraSize}" />
+	  </inertial>
+	</link>
 </robot>
