Commit message: enabled

File: mybot_description/urdf/macros.xacro (robot description, xacro)
@@ -51,5 +51,5 @@
 	  <parent link="chassis"/>
 	  <child link="${lr}_wheel"/>
-	<origin xyz="${-wheelPos+chassisLength/2} ${tY*wheelWidth/2+tY*chassisWidth/2} ${wheelRadius}" rpy="0 0 0" />
+	  <origin xyz="${-wheelPos+chassisLength/2} ${tY*wheelWidth/2+tY*chassisWidth/2} ${wheelRadius}" rpy="0 0 0" />
 	  <axis xyz="0 1 0" rpy="0 0 0" />
 	  <limit effort="100" velocity="100"/>
@@ -58,5 +58,7 @@
 	<transmission name="${lr}_trans">
 	  <type>transmission_interface/SimpleTransmission</type>
-	  <joint name="${lr}_wheel_hinge"/>
+	  <joint name="${lr}_wheel_hinge">
+          <hardwareInterface>EffortJointInterface</hardwareInterface>
+      </joint>
 	  <actuator name="${lr}Motor">
 	    <hardwareInterface>EffortJointInterface</hardwareInterface>
